File: hardware/BREAD_Slice.kicad_sch (KiCad schematic)
At the start: 15 parts, among them J1 Conn_01x10_Female, U1 AP63205

Commit message: review and revise board and update footprints
Parts:
- D1: footprint SparkFun-LED:WS2812-5050-4PIN -> KMLib_IC_SMD:WS2812-5050-4PIN
- HS1: footprint kml-custom:Thermal Pad -> KMLib_Mounting:Thermal Pad
Changed lines of the file:
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@@
 			)
 		)
-		(property "Footprint" "SparkFun-LED:WS2812-5050-4PIN"
+		(property "Footprint" "KMLib_IC_SMD:WS2812-5050-4PIN"
 			(at 13.97 49.53 0)
 			(effects
@@
 			)
 		)
-		(property "Footprint" "kml-custom:Thermal Pad"
+		(property "Footprint" "KMLib_Mounting:Thermal Pad"
 			(at 35.8648 97.79 0)
 			(effects
